File: Kicad/_autosave-AVMeter.sch (KiCad schematic (older format))
At the start: 62 parts, among them J1 Conn_01x16, J2 Screw_Terminal_01x02, J3 Screw_Terminal_01x02, J4 Screw_Terminal_01x02, J5 Screw_Terminal_01x03, J6 Conn_02x03_Odd_Even, J7 Conn_01x02, J8 Conn_01x02, U1 LT6105, U2 LT6105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

Commit message: added mount holes and other
Parts:
- added C21: 220nf, Capacitor_SMD:C_1206_3216Metric_Pad1.42x1.75mm_HandSolder, symbol AVMeter-rescue:C-Device
- C1, C10, C11, C12, C13, C14, C15, C16, C17, C18, C19, C2, C20, C3, C4, C5, C6, C7, C8, C9: symbol Device:C -> AVMeter-rescue:C-Device
- D1: symbol Reference_Voltage:LM4040DBZ-2.0 -> AVMeter-rescue:LM4040DBZ-2.0-Reference_Voltage
- D2: symbol pspice:DIODE -> AVMeter-rescue:DIODE-pspice
- J1: symbol Connector_Generic:Conn_01x16 -> AVMeter-rescue:Conn_01x16-Connector_Generic
- J2, J3, J4: symbol Connector:Screw_Terminal_01x02 -> AVMeter-rescue:Screw_Terminal_01x02-Connector
- J5: symbol Connector:Screw_Terminal_01x03 -> AVMeter-rescue:Screw_Terminal_01x03-Connector
- J6: symbol Connector_Generic:Conn_02x03_Odd_Even -> AVMeter-rescue:Conn_02x03_Odd_Even-Connector_Generic
- J7, J8: symbol Connector_Generic:Conn_01x02 -> AVMeter-rescue:Conn_01x02-Connector_Generic
- R1, R10, R11, R12, R13, R14, R15, R16, R19, R2, R20, R21, R22, R23, R24, R25, R26, R3, R4, R5, R6, R7, R8, R9: symbol Device:R -> AVMeter-rescue:R-Device
- RV1: symbol Device:R_POT_TRIM -> AVMeter-rescue:R_POT_TRIM-Device
- U4: symbol Amplifier_Operational:LM321 -> AVMeter-rescue:LM321-Amplifier_Operational
- U5: symbol Analog_ADC:MCP3208 -> AVMeter-rescue:MCP3208-Analog_ADC
- U7: symbol Regulator_Linear:L7805 -> AVMeter-rescue:L7805-Regulator_Linear
Connections:
- net -Vin: now also C21.1
- net GND: now also C21.2
